Commit message: zed_parser with zed model

File: jet_description/robots/fullbody.sldasm.urdf (robot description, URDF)
Before this commit: robot fullbody.sldasm, 30 links, 29 joints
Links:
- removed link world
- added link map
- added link zed_center; visual mesh filename=package://jet_description/meshes/ZED.stl
- added link zed_depth_camera
- added link zed_left_camera; visual cylinder length=.031 radius=0.007
- added link zed_right_camera; visual cylinder length=.031 radius=0.007
Joints:
- added joint zed_center_joint: type fixed, parent base_link, child zed_center, origin xyz=0.14739 0.0 0.66991 rpy=0 0 0
- added joint zed_depth_camera_joint: type fixed, parent zed_left_camera, child zed_depth_camera, origin xyz=0 0 0 rpy=-1.5707963267948966 0 -1.5707963267948966
- added joint zed_left_camera_joint: type fixed, parent zed_center, child zed_left_camera, origin xyz=0 0.06 0 rpy=0 0 0
- added joint zed_right_camera_joint: type fixed, parent zed_center, child zed_right_camera, origin xyz=0 -0.06 0 rpy=0 0 0
- joint virtual: axis (none) -> 0 0 1; parent world -> map; type fixed -> floating
